Commit message: Inertial Values fixed

File: phantomx_description/urdf/phantomx.ignition.xacro (robot description, xacro)
@@ -5,4 +5,18 @@
       <joint_name>j_thigh_${suffix}</joint_name>
       <joint_name>j_tibia_${suffix}</joint_name>
+    </xacro:macro>
+    <xacro:macro name="leg_colours" params="suffix">
+      <gazebo reference="c1_${suffix}">
+        <material>Gazebo/Grey</material>
+      </gazebo>
+      <gazebo reference="c2_${suffix}">
+        <material>Gazebo/Grey</material>
+      </gazebo>
+      <gazebo reference="thigh_${suffix}">
+        <material>Gazebo/Grey</material>
+      </gazebo>
+      <gazebo reference="tibia_${suffix}">
+        <material>Gazebo/Grey</material>
+      </gazebo>
     </xacro:macro>
     <xacro:macro name="phantomx_ign">
@@ -20,4 +34,10 @@
         <material>Gazebo/Grey</material>
       </gazebo>
+      <xacro:leg_colours suffix="lf"/>
+      <xacro:leg_colours suffix="rf"/>
+      <xacro:leg_colours suffix="lm"/>
+      <xacro:leg_colours suffix="rm"/>
+      <xacro:leg_colours suffix="lr"/>
+      <xacro:leg_colours suffix="rr"/>
       <gazebo>
         <plugin name="ignition::gazebo::systems::JointController" filename="ignition-gazebo-joint-controller-system">

File: phantomx_description/urdf/phantomx.xacro (robot description, xacro)
@@ -4,5 +4,5 @@
   <link name="base_link"/>
   <xacro:phantomx parent="base_link">
-      <origin xyz="0 0 0" rpy="0 0 0" />
+      <origin xyz="0 0 0.2" rpy="0 0 0" />
   </xacro:phantomx>
 </robot>

File: phantomx_description/urdf/phantomx_urdf.xacro (robot description, xacro)
@@ -49,5 +49,5 @@
         <origin xyz="0 -${connect_offset} 0" rpy="0 0 0"  />
         <mass value="0.024357719"/>
-       <inertia ixx="0.0051411124"  ixy="-0.00057530255"  ixz="-0.000024729049" iyy="0.0081915737" iyz="-0.000019223094" izz="0.0011379812" />
+        <inertia ixx="${(1/12)*(0.024357719)*((0.045)*(0.045) + (0.022)*(0.022))}"  ixy="0"  ixz="0" iyy="${(1/12)*(0.024357719)*((0.022)*(0.022) + (0.0325)*(0.0325))}" iyz="0" izz="${(1/12)*(0.024357719)*((0.0325)*(0.0325) + (0.045)*(0.045))}"/>
       </inertial>
       <visual>
@@ -72,5 +72,5 @@
         <origin xyz="0 -${connect_offset} 0" rpy="0 0 0"  />
         <mass value="0.024357719"/>
-       <inertia ixx="0.0051411124"  ixy="-0.00057530255"  ixz="-0.000024729049" iyy="0.0081915737" iyz="-0.000019223094" izz="0.0011379812" />
+        <inertia ixx="${(1/12)*(0.024357719)*((0.045)*(0.045) + (0.022)*(0.022))}"  ixy="0"  ixz="0" iyy="${(1/12)*(0.024357719)*((0.022)*(0.022) + (0.0325)*(0.0325))}" iyz="0" izz="${(1/12)*(0.024357719)*((0.0325)*(0.0325) + (0.045)*(0.045))}"/>
       </inertial>
       <visual>
@@ -95,5 +95,5 @@
         <origin xyz="0 0 0" rpy="0 0 0"  />
         <mass value="0.024357719"/>
-       <inertia ixx="0.0051411124"  ixy="-0.00057530255"  ixz="-0.000024729049" iyy="0.0081915737" iyz="-0.000019223094" izz="0.0011379812" />
+        <inertia ixx="${(1/12)*(0.024357719)*((0.045)*(0.045) + (0.022)*(0.022))}"  ixy="0"  ixz="0" iyy="${(1/12)*(0.024357719)*((0.022)*(0.022) + (0.0325)*(0.0325))}" iyz="0" izz="${(1/12)*(0.024357719)*((0.0325)*(0.0325) + (0.045)*(0.045))}"/>
       </inertial>
       <visual>
@@ -118,5 +118,5 @@
         <origin xyz="0 0 0" rpy="0 0 0"  />
         <mass value="0.024357719"/>
-       <inertia ixx="0.0051411124"  ixy="-0.00057530255"  ixz="-0.000024729049" iyy="0.0081915737" iyz="-0.000019223094" izz="0.0011379812" />
+        <inertia ixx="${(1/12)*(0.024357719)*((0.045)*(0.045) + (0.022)*(0.022))}"  ixy="0"  ixz="0" iyy="${(1/12)*(0.024357719)*((0.022)*(0.022) + (0.0325)*(0.0325))}" iyz="0" izz="${(1/12)*(0.024357719)*((0.0325)*(0.0325) + (0.045)*(0.045))}"/>
       </inertial>
       <visual>

Commit message: Trajectory Controller Implemented

File: phantomx_description/urdf/phantomx.ignition.xacro (robot description, xacro)
@@ -19,4 +19,11 @@
         <material>Gazebo/Grey</material>
       </gazebo>
+    </xacro:macro>
+    <xacro:macro name="pid">
+      <position_p_gain>3000</position_p_gain>
+      <position_d_gain>15</position_d_gain>
+      <position_i_gain>1650</position_i_gain>
+      <position_i_min>-15</position_i_min>
+      <position_i_max>15</position_i_max>
     </xacro:macro>
     <xacro:macro name="phantomx_ign">
@@ -41,5 +48,5 @@
       <xacro:leg_colours suffix="rr"/>
       <gazebo>
-        <plugin name="ignition::gazebo::systems::JointController" filename="ignition-gazebo-joint-controller-system">
+        <plugin name="ignition::gazebo::systems::JointTrajectoryController" filename="ignition-gazebo-joint-trajectory-controller-system">
           <xacro:leg_joints suffix="rf"/>
           <xacro:leg_joints suffix="lf"/>
@@ -48,4 +55,5 @@
           <xacro:leg_joints suffix="rr"/>
           <xacro:leg_joints suffix="lr"/>
+          <xacro:pid/>
         </plugin>
       </gazebo>
